File: phaseshiftfilter.kicad_sch (KiCad schematic)
At the start: 164 parts

Commit message: Upgrade
Connections:
- net F_IN is gone; now on net F_4: C100.1, C101.1, C102.1, C103.1, C104.1, C105.1, C106.1, C107.1, C69.1, C70.1, C71.1, C72.1, C73.1, C74.1, C75.1, C76.1, C77.1, C78.1, C79.1, C80.1, C81.1, C82.1, C83.1, C97.1, C98.1, C99.1, L1.3, L2.3, L2.4, L3.3, L3.4, L4.3, L4.4, L8.4
- net Line is gone; now on net F_CRC: C21.2, C22.2, C23.2, C24.2, C25.2, C26.2, C27.2, C58.2, C60.2, C62.2, C64.2, C66.2, C68.2, FL4.6, L11.1, L12.1
- net F_4: now also C108.1, C109.1, C110.1, C111.1, C35.2, C36.2, C37.2, C38.2, FL5.3, FL6.8, L1.4, L7.3
- net F_RC renamed F_CRC
Other:
- note added: "2024.12.03"
- note added: "7 devices by this this scheme at F_IN points to L and N"
- note added: "Notch filter at 30mkF and 10mkF,1mkF, 680nF, 100nF CRC filter to ground To L and N"
- note added: "Notch filter at 4mkF, 680 nF CRC filter to ground To L and N"
- note removed: "4 devices by this this scheme at F_IN points to L and N"
- note removed: "Notch filter at 30mkF and 10mkF RC filter to ground To L"
- note removed: "Notch filter at 4mkF CRC filter to ground To L and N"
Changed lines of the file:
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@@
 	)
 	(rectangle
-		(start 241.3225 137.4222)
-		(end 269.2625 156.4722)
+		(start 234.95 137.4222)
+		(end 276.86 156.4722)
 		(stroke
 			(width 0)
@@
 		)
 	)
-	(text "4 devices by this this scheme at F_IN points to L and N\n\n"
+	(text "7 devices by this this scheme at F_IN points to L and N\n\n"
 		(exclude_from_sim no)
 		(at 46.99 192.278 0)
@@
 		)
 	)
-	(text "Notch filter at\n4mkF \nCRC filter to ground\nTo L and N"
+	(text "Notch filter at\n4mkF, 680 nF \nCRC filter to ground\nTo L and N"
 		(exclude_from_sim no)
 		(at 208.28 147.32 0)
@@
 		)
 	)
+	(text "2024.12.03"
+		(exclude_from_sim no)
+		(at 263.906 178.816 0)
+		(effects
+			(font
+				(size 1.27 1.27)
+			)
+		)
+	)
 	(text "06.11.2024"
 		(exclude_from_sim no)
@@
 		)
 	)
-	(text "Notch filter at\n30mkF and 10mkF \nRC filter to ground\nTo L"
+	(text "Notch filter at\n30mkF and 10mkF,1mkF, 680nF, 100nF\nCRC filter to ground\nTo L and N"
 		(exclude_from_sim no)
 		(at 255.778 146.558 0)
@@
 		)
 	)
+	(global_label "F_IN"
+		(shape input)
+		(at 153.67 49.53 0)
+		(fields_autoplaced yes)
+		(effects
+			(font
+				(size 1.27 1.27)
+			)
+			(justify left)
+		)
+		(property "Intersheetrefs" "${INTERSHEET_REFS}"
+			(at 160.6467 49.53 0)
+			(effects
+				(font
+					(size 1.27 1.27)
+				)
+				(justify left)
+				(hide yes)
+			)
+		)
+	)
 	(global_label "C_30"
 		(shape input)
@@
 		)
 	)
-	(global_label "F_RC"
+	(global_label "F_IN"
+		(shape input)
+		(at 45.72 151.13 0)
+		(fields_autoplaced yes)
+		(effects
+			(font
+				(size 1.27 1.27)
+			)
+			(justify left)
+		)
+		(property "Intersheetrefs" "${INTERSHEET_REFS}"
+			(at 52.6967 151.13 0)
+			(effects
+				(font
+					(size 1.27 1.27)
+				)
+				(justify left)
+				(hide yes)
+			)
+		)
+	)
+	(global_label "F_CRC"
 		(shape input)
 		(at 252.73 139.7 0)
@@
 		)
 		(property "Intersheetrefs" "${INTERSHEET_REFS}"
-			(at 260.3114 139.7 0)
+			(at 261.5814 139.7 0)
 			(effects
 				(font
@@
 		)
 	)
+	(global_label "F_IN"
+		(shape input)
+		(at 104.14 49.53 0)
+		(fields_autoplaced yes)
+		(effects
+			(font
+				(size 1.27 1.27)
+			)
+			(justify left)
+		)
+		(property "Intersheetrefs" "${INTERSHEET_REFS}"
+			(at 111.1167 49.53 0)
+			(effects
+				(font
+					(size 1.27 1.27)
+				)
+				(justify left)
+				(hide yes)
+			)
+		)
+	)
 	(global_label "F_4"
 		(shape input)
@@
 		)
 	)
-	(global_label "F_RC"
+	(global_label "F_CRC"
 		(shape input)
 		(at 87.63 138.43 0)
@@
 		)
 		(property "Intersheetrefs" "${INTERSHEET_REFS}"
-			(at 95.2114 138.43 0)
+			(at 96.4814 138.43 0)
 			(effects
 				(font
@@
 			(effects
 				(font
+					(size 1.27 1.27)
+				)
+				(justify left)
+				(hide yes)
+			)
+		)
+	)
+	(global_label "F_CRC"
+		(shape input)
+		(at 172.72 158.75 0)
+		(fields_autoplaced yes)
+		(effects
+			(font
+				(size 1.27 1.27)
+			)
+			(justify left)
+		)
+		(property "Intersheetrefs" "${INTERSHEET_REFS}"
+			(at 181.5714 158.75 0)
+			(effects
+				(font

Commit message: Upgrade
Parts:
- removed C57, C58: 40nF, symbol Device:C
- removed C59, C60: 220pF, symbol Device:C
- removed C61, C62: 2.2nF, symbol Device:C
- removed C63, C64: 10nF, symbol Device:C
- removed C65, C66: 1nF, symbol Device:C
- removed C67, C68: 100pF, symbol Device:C
- removed L11, L12: 1:1 ~15 turns, symbol Device:L_Ferrite_Coupled
- removed R13, R16, R17, R18: 2, symbol Device:R
- removed R14, R15: 1, symbol Device:R
- added C128, C129: 1mkF, symbol Device:C
- C13: value 10mkF -> 1mkF
- L1: value Ferrite Transformer 1:1 ~10 turns -> Ferrite ST Transformer 1:1 ~20 turns
- L2: value Ferrite Transformer 5:1 where 1 is ~30 turns -> Ferrite Transformer with coupled coil 1:1 + 1:1 where 15 turns
- L3: value Ferrite Transformer 5:1 where 1 is ~30 turns -> Ferrite Transformer 5:1 where 1 is 5 turns
- L5: value 1:1 ~17 turns -> Ferrite CM choke 1:1 ~17 turns
- L6: value Ferrite Transformer 1:1 ~10 turns -> Ferrite CM choke 1:1 ~10 turns
- L8: value Ferrite Transformer 1:5 where 1 is 5 turns -> Ferrite Common mode 1:1 where 15 turns
- L9: value 1:1 ~20 turns -> CM 1:1 ~20 turns
Connections:
- net C_30: now also C21.2, C22.2, C23.2, C24.2, C25.2, C26.2, C27.2, C69.2, C70.2, C71.2, C72.2, C73.2, FL4.6, L2.1, L3.2; no longer C13.1
- net F_4: now also C13.2, C128.1, C128.2
- net Neutral: now also C10.2, C11.2, C12.2, C2.2, C4.2, C5.2, C52.2, C54.2, C56.2, C7.2, C8.2, C9.2, L9.3
- net at C108.2, C109.2, C110.2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: now also C129.2
- net at C35.1, C36.1, C37.1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: now also C13.1
- net F_CRC: no longer names the net of C100.2, C101.2, C102.2, C103.2, C104.2, C105.2, C106.2, C107.2, C97.2, C98.2, C99.2, L1.1, L2.2
- net F_CRC: now also C129.1; no longer C21.2, C22.2, C23.2, C24.2, C25.2, C26.2, C27.2, FL4.6

Commit message: Upgrade
Parts:
- added C130, C68: 2.2nF, symbol Device:C
- added C57: 10mkF, symbol Device:C
- added C58, C64, C65: 1mkF, symbol Device:C
- added C59: 500nF, symbol Device:C
- added C60: 100nF, symbol Device:C
- added C61: 40nF, symbol Device:C
- added C62: 10nF, symbol Device:C
- added C63: 1nF, symbol Device:C
- added C66, C67: 100 nF, symbol Device:C
- added RV1, RV2, RV3: Varistor, symbol Device:Varistor
- L3: value Ferrite Transformer 5:1 where 1 is 5 turns -> Ferrite Transformer 1:1 + 3:3 where 1 is 10 turns
- L4: value Ferrite Transformer 1:5 where 1 is 5 turns -> Ferrite Transformer 1:1 where 1 is 10 turns
Connections:
- net F_4 is gone; now on net C_30: C100.1, C101.1, C102.1, C103.1, C104.1, C105.1, C106.1, C107.1, C108.1, C109.1, C110.1, C111.1, C128.1, C128.2, C13.2, C35.2, C36.2, C37.2, C38.2, C69.1, C70.1, C71.1, C72.1, C73.1, C74.1, C75.1, C76.1, C77.1, C78.1, C79.1, C80.1, C81.1, C82.1, C83.1, C93.1, C94.1, C95.1, C96.1, C97.1, C98.1, C99.1, FL1.8, FL5.3, FL6.8, L1.3, L1.4, L2.3, L2.4, L3.3, L3.4, L4.3, L4.4, L5.3, L7.3, L8.4
- net C_30: now also C65.1, C65.2, C66.1, C66.2, C68.2, RV1.1, RV2.1, RV3.1; no longer C69.2, C70.2, C71.2, C72.2, C73.2, L2.1, L3.2
- net at C14.1, C15.1, C16.1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: now also C130.2
- net at C14.2, C15.2, C16.2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: now also C68.1
- net at C108.2, C109.2, C110.2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: now also C64.2, C67.2, RV1.2
- net at C100.2, C101.2, C102.2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: now also C64.1, C67.1, RV2.2
- net at C13.1, C35.1, C36.1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: now also C130.1
- new net: C57.1, C58.1, C59.1, C60.1, C61.1, C62.1, C63.1
- new net: C57.2, C58.2, C59.2, C60.2, C61.2, C62.2, C63.2
- new net: C69.2, C70.2, C71.2, C72.2, C73.2, L2.1, L3.2, RV3.2
Other:
- note added: "EMC block"
- note added: "LOAD 1"
- note added: "LOAD 2"
- note added: "Notch filter at 10mkF,1mkF, 680nF, 100nF CRC filter to ground To L and N"
- note added: "Notch filter at 4mkF, 680 nF, 1mkF CRC filter to ground To L and N"
- note added: "Notch filters at 30 mkF. 80 mkF, 800 mkF CRC To L and N"
- note removed: "Notch filter at 30mkF and 10mkF,1mkF, 680nF, 100nF CRC filter to ground To L and N"
- note removed: "Notch filter at 4mkF, 680 nF CRC filter to ground To L and N"

Commit message: Upgrade
Parts:
- added C131: 1mkF, symbol Device:C
- added C132: 10nF, symbol Device:C
- added K1: Relay_SPDT, symbol Relay:Relay_SPDT
- added L10: CM 1:1 ~4-8 turns, symbol Device:L_Ferrite_Coupled
- added R13, R14: 680kOm, symbol Device:R
- L7: value 1:1 ~12 turns -> 1:1 ~4-8 turns
- L9: value CM 1:1 ~20 turns -> CM 1:1 ~4-8 turns
Connections:
- net C_30: now also C74.2, C75.2, C76.2, C77.2, C78.2, L3.1, L4.2, C131.1, C132.1, K1.11, L10.1, R13.2, R14.2
- net Neutral: now also L10.3
- net at C130.2, C14.1, C15.1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: now also L10.2
- net at C14.2, C15.2, C16.2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: now also L10.4
- new net: C132.2, K1.14, R14.1
- new net: C131.2, K1.12, R13.1
Other:
- note added: "And, by the using GD logic with releys, swith pair of capacitors from 105 to 103"
- note added: "Filter With Capacitor Switch"
- note removed: "Filter With Phase Shift"

Commit message: Upgrade
Parts:
- RV1, RV2, RV3: value Varistor -> ~230-240V
Changed lines of the file:
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@@
 			)
 		)
-		(property "Value" "Varistor"
+		(property "Value" "~230-240V"
 			(at 39.5633 149.86 90)
 			(effects
@@
 		(on_board yes)
 		(dnp no)
-		(fields_autoplaced yes)
 		(property "Reference" "RV2"
-			(at 39.5633 125.73 90)
+			(at 39.37 123.444 90)
 			(effects
 				(font
@@
 			)
 		)
-		(property "Value" "Varistor"
-			(at 39.5633 128.27 90)
+		(property "Value" "~230-240V"
+			(at 38.354 126.238 90)
 			(effects
 				(font
@@
 			)
 		)
-		(property "Value" "Varistor"
+		(property "Value" "~230-240V"
 			(at 39.5633 110.49 90)
 			(effects

Commit message: Upgrade
Parts:
- L10: value CM 1:1 ~4-8 turns -> CM 1:1 ~4-8 turns Optional
Connections:
- net SwitchingCapacitorsIn1: now reaches FL1.1, L7.2
- net SwitchingCapacitorsIn2: now reaches C120.1, C121.1, C122.1, C123.1, FL3.8, FL4.3

Commit message: Upgrade
Parts:
- removed C1, C106, C132, C19, C2, C33, C35, C41, C42, C47, C48, C8, C95: 10nF, symbol Device:C
- removed C10, C104, C17, C31, C38: 100nF, symbol Device:C
- removed C105, C18, C32, C37, C51, C52, C9: 40nF, symbol Device:C
- removed C107, C20, C3, C34, C36, C4, C43, C44, C49, C50, C7, C96: 1nF, symbol Device:C
- removed C11, C16, C30: 500nF, symbol Device:C
- removed C12, C13, C15, C29, C64, C65: 1mkF, symbol Device:C
- removed C14, C28: 10mkF, symbol Device:C
- removed C39, C40, C45, C46, C5, C6: 82nF, symbol Device:C
- removed C53, C54: 220pF, symbol Device:C
- removed C55, C56, C68: 2.2nF, symbol Device:C
- removed C66, C67: 100 nF, symbol Device:C
- removed FL1, FL6: 4-6 turns on each coil at choke Ferrite, symbol Device:Filter_EMI_LLLL
- removed K1: Relay_SPDT, symbol Relay:Relay_SPDT
- removed L10: CM 1:1 ~4-8 turns Optional, symbol Device:L_Ferrite_Coupled
- removed L5: Ferrite CM choke 1:1 ~17 turns, symbol Device:L_Ferrite_Coupled
- removed L6: Ferrite CM choke 1:1 ~10 turns, symbol Device:L_Ferrite_Coupled
- removed L7: 1:1 ~4-8 turns, symbol Device:L_Ferrite_Coupled
- removed L9: CM 1:1 ~4-8 turns, symbol Device:L_Ferrite_Coupled
- removed R10, R7, R8, R9: 2, symbol Device:R
- removed R11, R12: 1, symbol Device:R
- removed R13, R14: 680kOm, symbol Device:R
- added RV4, RV5, RV6: ~230-240V, symbol Device:Varistor
- C128, C129, C131: value 1mkF -> 10mkF
- C130: value 2.2nF -> 10mkF
- C89, C93: value 100nF -> 100 nF
- C90, C94: value 1mkF -> 100 nF
- C91: value 10nF -> 100 nF
- C92: value 1nF -> 100 nF
- C97: value 500nF -> 22nF
- L1: value Ferrite ST Transformer 1:1 ~20 turns -> Ferrite Choke 1:1 ~20 turns
- L2: value Ferrite Transformer with coupled coil 1:1 + 1:1 where 15 turns -> Ferrite double core choke with coupled coil 1:1 + 1:1 where 15 turns
- L3: value Ferrite Transformer 1:1 + 3:3 where 1 is 10 turns -> Ferrite double core choke with coupled coil 1:1 + 1:1 where 15 turns
- L4: value Ferrite Transformer 1:1 where 1 is 10 turns -> Ferrite double core choke with coupled coil 1:1 + 1:1 where 15 turns
- L8: value Ferrite Common mode 1:1 where 15 turns -> UHF Ferrite Common mode 1:1 where 4 turns
- R1, R2, R3, R4, R5, R6: value 2 -> 220 R
Connections:
- net C_30: now also C129.1, C130.1, C130.2, C79.2, C80.2, C81.2, C82.2, C83.2, C84.1, C85.1, C86.1, C87.1, C88.1, C90.1, C91.1, C92.1, L4.1, L8.2, L8.3, R3.2, RV4.1, RV5.1, RV5.2, RV6.1; no longer C108.1, C109.1, C110.1, C111.1, C128.2, C74.2, C75.2, C76.2, C77.2, C78.2, FL5.3, L1.4, L3.1, L4.2, RV1.1
- net C_910: now also C108.2, C109.2, C110.2, C111.2, FL5.3, L1.2, R1.2, RV1.2
- net Earth: no longer R1.2, R2.2, R3.2, R4.2, R5.2, R6.2
- net Neutral: now also C131.2, C84.2, C85.2, C86.2, C87.2, C88.2, L8.1, R2.2, RV6.2
- net at C100.2, C101.2, C102.2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: now also R6.2; no longer C129.1
- net at R1.1: now also C89.2
- net at R4.1: now also C92.2
- net at R2.1: now also C90.2
- net at C93.2: now also R5.1; no longer C94.2
- net at C69.2, C70.2, C71.2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: now also C128.2, R5.2
- net at R3.1: now also C91.2
- net at R6.1: now also C94.2
- net SwitchingCapacitorsIn2: no longer names the net of C120.1, C121.1, C122.1, C123.1, FL3.8, FL4.3
- new net: C108.1, C109.1, C110.1, C111.1, C89.1, FL5.1, L1.4, RV1.1
- new net: C129.2, C74.2, C75.2, C76.2, C77.2, C78.2, L3.1, L4.2, R4.2, RV4.2
Other:
- note added: "Notch filters at 1mkF, 10 mkF, 30 mkF. 80 mkF, 800 mkF CRC To L and N"
- note removed: "And, by the using GD logic with releys, swith pair of capacitors from 105 to 103"
- note removed: "Notch filters at 30 mkF. 80 mkF, 800 mkF CRC To L and N"

Commit message: Upgrade
Parts:
- removed C21, C57: 10mkF, symbol Device:C
- removed C22, C58: 1mkF, symbol Device:C
- removed C23, C59: 500nF, symbol Device:C
- removed C24, C60: 100nF, symbol Device:C
- removed C25, C61: 40nF, symbol Device:C
- removed C26, C62: 10nF, symbol Device:C
- removed C27, C63: 1nF, symbol Device:C
- removed FL4: 4-6 turns on each coil at choke Ferrite, symbol Device:Filter_EMI_LLLL
- added C104, C95, C96: 100 nF, symbol Device:C
- added R7, R8, R9: 220 R, symbol Device:R
- added RV7, RV8, RV9: ~230-240V, symbol Device:Varistor
- L1: value Ferrite Choke 1:1 ~20 turns -> Ferrite double core choke with coupled coil 1:1 + 1:1 where 15 turns
Connections:
- net Neutral is gone; now on net C_910: C131.2, C84.2, C85.2, C86.2, C87.2, C88.2, L8.1, R2.2, RV6.2
- net C_30: now also C104.1, RV7.1
- net C_910: now also C120.1, C121.1, C122.1, C123.1, FL3.8, R9.2, RV7.2
- net To Load 1: now reaches C108.1, C109.1, C110.1, C111.1, C89.1, FL5.1, L1.4, RV1.1
- net at C112.1, C113.1, C114.1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: now also C95.1, RV9.2
- net at C112.2, C113.2, C114.2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: now also R7.2, RV9.1
- net at C116.1, C117.1, C118.1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: now also C96.1, RV8.2
- net at C116.2, C117.2, C118.2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: now also R8.2, RV8.1
- new net: C96.2, R8.1
- new net: C104.2, R9.1
- new net: C95.2, R7.1
Other:
- note added: "2025.04.22"
- note added: "Do not power on illumination from any outputs for load"
- note added: "Use 2 or 3 ground device with switched resistors for ground filters trought one"
