File: phaseshiftfilter.kicad_sch (KiCad schematic)
At the start: 88 parts

Commit message: Update
Parts:
- removed C100, C111, C115, C119, C123, C72: 10nF, symbol Device:C
- removed C101, C128: 10mkF, symbol Device:C
- removed C102, C110, C114, C118, C122, C71, C99: 1mkF, symbol Device:C
- removed C103, C108, C112, C116, C120, C69: 500nF, symbol Device:C
- removed C104, C89, C90, C91, C92, C93, C94, C95, C96: 100 nF, symbol Device:C
- removed C109, C113, C117, C121, C70, C98: 100nF, symbol Device:C
- removed C73: 1nF, symbol Device:C
- removed C97: 22nF, symbol Device:C
- removed FL2, FL3, FL5: 4-6 turns on each coil at choke Ferrite, symbol Device:Filter_EMI_LLLL
- removed L1, L2, L3: Ferrite double core choke with coupled coil 1:1 +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, symbol Device:L_Ferrite_Coupled
- removed R1, R2, R3, R4, R5, R6, R7, R8, R9: 220 R, symbol Device:R
- removed R19, R20: 1, symbol Device:R
- removed RV1, RV2, RV3, RV7, RV8, RV9: ~230-240V, symbol Device:Varistor
- added C1, C2: 100pF, symbol Device:C
- added C10, C9: 1nF, symbol Device:C
- added C11, C12: 330pF, symbol Device:C
- added C13, C14: 150pF, symbol Device:C
- added C15, C16: 3.3nF, symbol Device:C
- added C17, C18: 4.7nF, symbol Device:C
- added C19: 5.6pF, symbol Device:C
- added C20: 5.6nF, symbol Device:C
- added C21, C22: 6.8nF, symbol Device:C
- added C23, C24: 8.2nF, symbol Device:C
- added C25, C26: 10nF, symbol Device:C
- added C27, C28, C29: 2.2mkF, symbol Device:C
- added C3, C4: 680pF, symbol Device:C
- added C5, C6: 470pF, symbol Device:C
- added C7, C8: 820pF, symbol Device:C
- C126, C127: value 2.2nF -> 560pF
- L8: value UHF Ferrite Common mode 1:1 where 4 turns -> UHF Ferrite Common mode 1:1 where 2 turns
Connections:
- net C_910 is gone; now on net C_30: C131.2, C84.2, C85.2, C86.2, C87.2, C88.2, L8.1, RV6.2
- net C_30: now also C27.1, C28.1, C28.2, C29.1, C29.2
- net Earth: now also C124.2, C125.1, C126.2, C127.1, C1.2, C10.1, C11.2, C12.1, C13.2, C14.1, C15.2, C16.1, C17.2, C18.1, C19.2, C2.1, C20.1, C21.2, C22.1, C23.2, C24.1, C25.2, C26.1, C3.2, C4.1, C5.2, C6.1, C7.2, C8.1, C9.2
- net at C129.2, C74.2, C75.2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: now also C27.2
- net at C124.1, C126.1: now also C1.1, C11.1, C13.1, C16.2, C18.2, C20.2, C22.2, C24.2, C26.2, C3.1, C5.1, C7.1, C9.1
- net at C125.2, C127.2: now also C10.2, C12.2, C14.2, C15.1, C17.1, C19.1, C2.2, C21.1, C23.1, C25.1, C4.2, C6.2, C8.2
Other:
- note added: "3 devices by this this scheme at F_IN points to L and N"
- note added: "Do not builded because of problems with money"
- note added: "Notch filter at 2-6mkF,1mkF, 680nF, 100nF X/Y filter to ground To L and N"
- note added: "Notch filter at 4mkF, 680 nF, 1mkF X/Y filter to ground To L and N"
- note added: "Notch filters at 1mkF, 10 mkF. 80 mkF, 800 mkF X/Y To L and N"
- note added: "Notch filters at 30 mkF X/Y capacitor To L and N"
- note removed: "7 devices by this this scheme at F_IN points to L and N"
- note removed: "EMC block"
- note removed: "Notch filter at 10mkF,1mkF, 680nF, 100nF CRC filter to ground To L and N"
- note removed: "Notch filter at 4mkF, 680 nF, 1mkF CRC filter to ground To L and N"
- note removed: "Notch filters at 1mkF, 10 mkF, 30 mkF. 80 mkF, 800 mkF CRC To L and N"
- note removed: "Notch filters at 30 mkF capacitor To L and N"
- moved on the sheet: C129, C74, C75, C76, C77, C78
